File: ab-mix/1_Input.sch (KiCad schematic (older format))
At the start: 34 parts, among them Q1 J201, Q2 J201, SW1 SW_SPST, SW2 SW_Push_3PDT, U1 LM324, U2 CD4053B

Commit message: Placed Jacks and Switches
Parts:
- removed SW1: SW_SPST, MBv3 switches:SPST.WIRE, symbol Switch:SW_SPST
- added H1: Flip1, pedal-component-footprint:PinHeader_1x01_P2.54mm_Vertical_Front_Back, symbol Mechanical:MountingHole_Pad
- added H2: Flip2, pedal-component-footprint:PinHeader_1x01_P2.54mm_Vertical_Front_Back, symbol Mechanical:MountingHole_Pad
- SW1: renamed from SW2; value SW_Push_3PDT -> Phase
Connections:
- net GND: now also H2.1
- net at R7.1, R8.2: now also H1.1
Changed lines of the file:
@@
 	2450 4725 2900 4725
 $Comp
-L Switch:SW_Push_3PDT SW2
+L Switch:SW_Push_3PDT SW1
 U 1 1 5FBD9FFB
 P 8350 5650
-F 0 "SW2" H 8350 6335 50  0000 C CNN
-F 1 "SW_Push_3PDT" H 8350 6244 50  0000 C CNN
+F 0 "SW1" H 8350 6335 50  0000 C CNN
+F 1 "Phase" H 8350 6244 50  0000 C CNN
 F 2 "pedal-component-footprint:3PDT.LUGS.FLPVSK" H 8350 6010 50  0001 C CNN
 F 3 "~" H 8350 6010 50  0001 C CNN
@@
 	1    0    0    1
 $EndComp
-Text GLabel 9100 6050 3    50   Input ~ 0
-+4V5
 $Comp
 L Device:LED D1
@@
 U 1 1 5FD38FD5
 P 9600 1550
-F 0 "R19" H 9750 1500 50  0000 R CNN
+F 0 "R19" H 9800 1475 50  0000 R CNN
 F 1 "1M" H 9800 1600 50  0000 R CNN
 F 2 "MBv3 resistors:0.3_22.B" V 9530 1550 50  0001 C CNN
@@
 	1    0    0    -1
 $EndComp
-$Comp
-L Switch:SW_SPST SW1
-U 1 1 5FC2D81E
-P 5100 2050
-F 0 "SW1" H 5100 2285 50  0000 C CNN
-F 1 "SW_SPST" H 5100 2194 50  0000 C CNN
-F 2 "MBv3 switches:SPST.WIRE" H 5100 2050 50  0001 C CNN
-F 3 "~" H 5100 2050 50  0001 C CNN
-	1    5100 2050
-	0    1    1    0
-$EndComp
 Wire Wire Line
 	5100 1200 5100 1300
@@
 Wire Wire Line
 	4725 7125 4725 6900
+Wire Wire Line
+	4725 6125 4725 6300
+Text GLabel 9100 6050 3    50   Input ~ 0
++4V5
 Text GLabel 4725 6125 1    50   Input ~ 0
 +9V
-Wire Wire Line
-	4725 6125 4725 6300
+$Comp
+L Mechanical:MountingHole_Pad H1
+U 1 1 5FDD123A
+P 4825 1850
+F 0 "H1" V 5050 1900 50  0000 C CNN
+F 1 "Flip1" V 4975 1900 50  0000 C CNN
+F 2 "pedal-component-footprint:PinHeader_1x01_P2.54mm_Vertical_Front_Back" H 4825 1850 50  0001 C CNN
+F 3 "~" H 4825 1850 50  0001 C CNN
+	1    4825 1850
+	0    -1   -1   0
+$EndComp
+$Comp
+L Mechanical:MountingHole_Pad H2
+U 1 1 5FDD1CCA
+P 4825 2250
+F 0 "H2" V 5050 2300 50  0000 C CNN
+F 1 "Flip2" V 4975 2300 50  0000 C CNN
+F 2 "pedal-component-footprint:PinHeader_1x01_P2.54mm_Vertical_Front_Back" H 4825 2250 50  0001 C CNN
+F 3 "~" H 4825 2250 50  0001 C CNN
+	1    4825 2250
+	0    -1   -1   0
+$EndComp
+Wire Wire Line
+	4925 2250 5100 2250
+Wire Wire Line
+	4925 1850 5100 1850
 $EndSCHEMATC

Commit message: That LAST connection!
Parts:
- C1, C5, C6: footprint MBv3 caps-film:0.2%22.MED -> MBv3 caps-film:0.2%22.SML
- C2, C3: value .1u -> 1u
Changed lines of the file:
@@
 F 0 "C1" V 1702 2775 50  0000 C CNN
 F 1 ".1u" V 1611 2775 50  0000 C CNN
-F 2 "MBv3 caps-film:0.2%22.MED" H 1450 2775 50  0001 C CNN
+F 2 "MBv3 caps-film:0.2%22.SML" H 1450 2775 50  0001 C CNN
 F 3 "~" H 1450 2775 50  0001 C CNN
 	1    1450 2775
@@
 P 2850 3025
 F 0 "C2" V 3102 3025 50  0000 C CNN
-F 1 ".1u" V 3011 3025 50  0000 C CNN
+F 1 "1u" V 3011 3025 50  0000 C CNN
 F 2 "MBv3 caps-film:0.2%22.MED" H 2850 3025 50  0001 C CNN
 F 3 "~" H 2850 3025 50  0001 C CNN
@@
 P 3050 4725
 F 0 "C3" V 3302 4725 50  0000 C CNN
-F 1 ".1u" V 3211 4725 50  0000 C CNN
+F 1 "1u" V 3211 4725 50  0000 C CNN
 F 2 "MBv3 caps-film:0.2%22.MED" H 3050 4725 50  0001 C CNN
 F 3 "~" H 3050 4725 50  0001 C CNN
@@
 F 0 "C5" V 6552 4350 50  0000 C CNN
 F 1 ".1u" V 6461 4350 50  0000 C CNN
-F 2 "MBv3 caps-film:0.2%22.MED" H 6300 4350 50  0001 C CNN
+F 2 "MBv3 caps-film:0.2%22.SML" H 6300 4350 50  0001 C CNN
 F 3 "~" H 6300 4350 50  0001 C CNN
 	1    6300 4350
@@
 F 0 "C6" V 6552 5550 50  0000 C CNN
 F 1 ".1u" V 6461 5550 50  0000 C CNN
-F 2 "MBv3 caps-film:0.2%22.MED" H 6300 5550 50  0001 C CNN
+F 2 "MBv3 caps-film:0.2%22.SML" H 6300 5550 50  0001 C CNN
 F 3 "~" H 6300 5550 50  0001 C CNN
 	1    6300 5550
