File: ab-mix/2_Crossfader_Hardware.sch (KiCad schematic (older format))
At the start: 28 parts, among them J1 IN, J2 Out, J3 Jack-DC, J4 Send1, J5 Return1, J6 Send2, J7 Return2, J8 Exp, Q3 Q_PNP_EBC, U3 LM324, U4 LM13700

Commit message: Placed Jacks and Switches
Parts:
- removed J3: Jack-DC, symbol Connector:Jack-DC
- added D4: Bypass, MBv3 diodes:3MM_1, symbol Device:LED
- added H3: 9V, pedal-component-footprint:PinHeader_1x01_P2.54mm_Vertical_Front_Back, symbol Mechanical:MountingHole_Pad
- added H4: GND, pedal-component-footprint:PinHeader_1x01_P2.54mm_Vertical_Front_Back, symbol Mechanical:MountingHole_Pad
- added H5: CV_DEFAULT, pedal-component-footprint:PinHeader_1x01_P2.54mm_Vertical_Front_Back, symbol Mechanical:MountingHole_Pad
- added R30: Rled, MBv3 resistors:0.3_22.B, symbol Device:R
- added RV2: 5K, MBv3 potentiometers:TRIM1, symbol Device:R_POT_TRIM
- added SW2: Bypass, pedal-component-footprint:3PDT.LUGS.FLPVSK, symbol Switch:SW_Push_3PDT
- J1, J2: footprint (none) -> pedal-component-footprint:Jack_6.35mm_Neutrik_NMJ6HCD3_Horizontal; symbol Connector:AudioJack3 -> Connector:AudioJack3_Switch
- J3: renamed from J4; footprint (none) -> pedal-component-footprint:Jack_6.35mm_Neutrik_NMJ6HCD3_Horizontal; symbol Connector:AudioJack3 -> Connector:AudioJack3_Switch
- J4: renamed from J5; footprint (none) -> pedal-component-footprint:Jack_6.35mm_Neutrik_NMJ6HCD3_Horizontal; symbol Connector:AudioJack3 -> Connector:AudioJack3_Switch
- J5: renamed from J6; footprint (none) -> pedal-component-footprint:Jack_6.35mm_Neutrik_NMJ6HCD3_Horizontal; symbol Connector:AudioJack3 -> Connector:AudioJack3_Switch
- J6: renamed from J7; footprint (none) -> pedal-component-footprint:Jack_6.35mm_Neutrik_NMJ6HCD3_Horizontal; symbol Connector:AudioJack3 -> Connector:AudioJack3_Switch
- J7: renamed from J8; footprint (none) -> pedal-component-footprint:Jack_6.35mm_Neutrik_NMJ6HCD3_Horizontal; symbol Connector:AudioJack3 -> Connector:AudioJack3_Switch
- RV1: value R_POT_TRIM -> 10K
- renumbered R30 to R31, R31 to R32, RV2 to RV3
Connections:
- net FX_RETURN1: no longer J4.R
- net FX_RETURN2: no longer J6.R
- net FX_SEND1: no longer J3.R
- net FX_SEND2: no longer J5.R
- net GND: now also J1.S, J1.SN, J2.S, J2.SN, J3.S, J3.SN, J4.S, J4.SN, J5.S, J5.SN, J6.S, J6.SN, H4.1, RV2.1, SW2.2 (B), SW2.3 (C), SW2.6 (C)
- net IN: now also SW2.5 (B); no longer J1.R, J1.T
- net OUT: now also SW2.7 (A); no longer J2.R, J2.T
- net 4V5 renamed +4V5
- net 9V renamed +9V
- net +9V: now also D4.2 (A), H3.1
- new net: H5.1, J7.TN
- new net: J7.S, RV2.2
- new net: R30.2, SW2.1 (A)
- new net: D4.1 (K), R30.1
- new net JACK_IN: J1.T, SW2.4 (A), SW2.9 (C)
- new net JACK_OUT: J2.T, SW2.8 (B)
- no-connect marks 15 -> 36

Commit message: That LAST connection!
Parts:
- C9: footprint MBv3 caps-film:0.2%22.LRG -> MBv3 caps-film:0.2%22.MED
- RV3: value R_POT -> Volume
Changed lines of the file:
@@
 F 0 "C9" V 9198 1650 50  0000 C CNN
 F 1 "1u" V 9289 1650 50  0000 C CNN
-F 2 "MBv3 caps-film:0.2%22.LRG" H 9488 1500 50  0001 C CNN
+F 2 "MBv3 caps-film:0.2%22.MED" H 9488 1500 50  0001 C CNN
 F 3 "~" H 9450 1650 50  0001 C CNN
 	1    9450 1650
@@
 P 10300 1900
 F 0 "RV3" H 10231 1854 50  0000 R CNN
-F 1 "R_POT" H 10231 1945 50  0000 R CNN
+F 1 "Volume" H 10231 1945 50  0000 R CNN
 F 2 "MBv3 potentiometers:16MM_B.MOUNT" H 10300 1900 50  0001 C CNN
 F 3 "~" H 10300 1900 50  0001 C CNN
