File: ab-mix/ab-mix.kicad_pcb (KiCad board)
At the start: 2 copper layers, 70 parts, among them J1 IN, J2 Out, J3 Send1, J4 Return1, J5 Send2, J6 Return2, J7 Exp, Q1 J201, Q2 J201, Q3 Q_PNP_EBC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

Commit message: All jacks and the pot placed
Parts:
- moved RV3 205.5 mm to (149.0, 68.5), turned to 90 degrees
- moved J7 193.5 mm to (85.0, 73.5), turned to 90 degrees
- moved J2 169.4 mm to (119.5, 73.5), turned to 90 degrees
- moved J1 149.8 mm to (64.0, 73.5), turned to 90 degrees
Changed lines of the file:
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@@
   )
   (module "MBv3 potentiometers:16MM_B.MOUNT" (layer F.Cu)
-    (at -50.4887 117.7943)
+    (at 149 68.5 90)
     (descr "<b>16mm / Right-Angle /  PC Mount / Short Pin</b>\n<p>\nFor bottom-mount potentiometers\n<p>\n<a href=\"http://smallbear-electronics.mybigcommerce.com/alpha-single-gang-16mm-right-angle-pc-mount/\">http://smallbear-electronics.mybigcommerce.com/alpha-single-gang-16mm-right-angle-pc-mount/</a>")
-    (fp_text reference RV3 (at 0 -2.413) (layer B.SilkS)
+    (fp_text reference RV3 (at 0 -2.413 90) (layer B.SilkS)
       (effects (font (size 1.2065 1.2065) (thickness 0.1524)) (justify mirror))
     )
-    (fp_text value R_POT (at -0.0635 -2.3495) (layer F.SilkS)
+    (fp_text value R_POT (at -0.0635 -2.3495 90) (layer F.SilkS)
       (effects (font (size 1 1) (thickness 0.15)))
     )
@@
     (fp_line (start -8.89 -14.605) (end 8.89 -14.605) (layer B.SilkS) (width 0.127))
     (fp_line (start -7.62 -1.651) (end 7.62 -1.651) (layer B.SilkS) (width 0.127))
-    (fp_text user 1 (at 6.35 -2.032) (layer F.SilkS)
+    (fp_text user 1 (at 6.35 -2.032 90) (layer F.SilkS)
       (effects (font (size 0.77216 0.77216) (thickness 0.097536)))
     )
@@
     (fp_line (start 3.556 1.524) (end 6.604 1.524) (layer B.SilkS) (width 0.127))
     (fp_line (start 6.604 1.524) (end 6.604 -1.524) (layer B.SilkS) (width 0.127))
-    (pad 1 thru_hole rect (at 5.08 0 180) (size 2.54 2.54) (drill 1.4) (layers *.Cu *.Mask)
-      (net 7 GND))
-    (pad 2 thru_hole oval (at 0 0 180) (size 2.54 2.54) (drill 1.4) (layers *.Cu *.Mask)
+    (pad 1 thru_hole rect (at 5.08 0 270) (size 2.54 2.54) (drill 1.4) (layers *.Cu *.Mask)
+      (net 7 GND))
+    (pad 2 thru_hole oval (at 0 0 270) (size 2.54 2.54) (drill 1.4) (layers *.Cu *.Mask)
       (net 69 OUT))
-    (pad 3 thru_hole oval (at -5.08 0 180) (size 2.54 2.54) (drill 1.4) (layers *.Cu *.Mask)
+    (pad 3 thru_hole oval (at -5.08 0 270) (size 2.54 2.54) (drill 1.4) (layers *.Cu *.Mask)
       (net 66 "Net-(R32-Pad1)"))
   )
@@
   )
   (module pedal-component-footprint:Jack_6.35mm_Neutrik_NMJ6HCD3_Horizontal (layer F.Cu)
-    (at -108.5172 74.9808)
+    (at 85 73.5 90)
     (descr "M Series, 6.35mm (1/4in) stereo jack, switched, with chrome ferrule and offset PCB pins, https://www.neutrik.com/en/product/nmj6hcd3")
     (tags "neutrik jack m")
-    (fp_text reference J7 (at 6.35 6.0325) (layer F.Fab)
-      (effects (font (size 1 1) (thickness 0.15)))
-    )
-    (fp_text value Exp (at 5.3975 7.874) (layer B.SilkS)
+    (fp_text reference J7 (at 6.35 6.0325 90) (layer F.Fab)
+      (effects (font (size 1 1) (thickness 0.15)))
+    )
+    (fp_text value Exp (at 5.3975 7.874 90) (layer B.SilkS)
       (effects (font (size 1 1) (thickness 0.15)) (justify mirror))
     )
-    (fp_text user %V (at 5.7 7.9) (layer F.SilkS)
+    (fp_text user %V (at 5.7 7.9 90) (layer F.SilkS)
       (effects (font (size 1 1) (thickness 0.15)))
     )
@@
     (fp_line (start -5.48 3.645) (end -5.48 -1.105) (layer B.SilkS) (width 0.12))
     (fp_line (start 15.37 2.295) (end 15.37 -1.105) (layer B.SilkS) (width 0.12))
-    (pad R thru_hole circle (at 6.35 0) (size 3.2 3.2) (drill 1.7) (layers *.Cu *.Mask)
+    (pad R thru_hole circle (at 6.35 0 90) (size 3.2 3.2) (drill 1.7) (layers *.Cu *.Mask)
       (net 13 +9V))
-    (pad S thru_hole circle (at 12.7 0) (size 3.2 3.2) (drill 1.7) (layers *.Cu *.Mask)
+    (pad S thru_hole circle (at 12.7 0 90) (size 3.2 3.2) (drill 1.7) (layers *.Cu *.Mask)
       (net 44 "Net-(J7-PadS)"))
-    (pad T thru_hole circle (at 0 0) (size 3.2 3.2) (drill 1.7) (layers *.Cu *.Mask)
+    (pad T thru_hole circle (at 0 0 90) (size 3.2 3.2) (drill 1.7) (layers *.Cu *.Mask)
       (net 45 CV))
-    (pad RN thru_hole circle (at 6.35 16.23) (size 3.2 3.2) (drill 1.7) (layers *.Cu *.Mask)
+    (pad RN thru_hole circle (at 6.35 16.23 90) (size 3.2 3.2) (drill 1.7) (layers *.Cu *.Mask)
       (net 46 "Net-(J7-PadRN)"))
-    (pad SN thru_hole circle (at 12.7 16.23) (size 3.2 3.2) (drill 1.7) (layers *.Cu *.Mask)
+    (pad SN thru_hole circle (at 12.7 16.23 90) (size 3.2 3.2) (drill 1.7) (layers *.Cu *.Mask)
       (net 47 "Net-(J7-PadSN)"))
-    (pad TN thru_hole circle (at 0 16.23) (size 3.2 3.2) (drill 1.7) (layers *.Cu *.Mask)
+    (pad TN thru_hole circle (at 0 16.23 90) (size 3.2 3.2) (drill 1.7) (layers *.Cu *.Mask)
       (net 23 "Net-(H5-Pad1)"))
     (model ${KISYS3DMOD}/Connector_Audio.3dshapes/Jack_6.35mm_Neutrik_NMJ6HCD3_Horizontal.wrl
@@
   )
   (module pedal-component-footprint:Jack_6.35mm_Neutrik_NMJ6HCD3_Horizontal (layer F.Cu)
-    (at -49.9172 74.9808)
+    (at 119.5 73.5 90)
     (descr "M Series, 6.35mm (1/4in) stereo jack, switched, with chrome ferrule and offset PCB pins, https://www.neutrik.com/en/product/nmj6hcd3")
     (tags "neutrik jack m")
-    (fp_text reference J2 (at 6.35 6.0325) (layer F.Fab)
-      (effects (font (size 1 1) (thickness 0.15)))
-    )
-    (fp_text value Out (at 5.3975 7.874) (layer B.SilkS)
+    (fp_text reference J2 (at 6.35 6.0325 90) (layer F.Fab)
+      (effects (font (size 1 1) (thickness 0.15)))
+    )
+    (fp_text value Out (at 5.3975 7.874 90) (layer B.SilkS)
       (effects (font (size 1 1) (thickness 0.15)) (justify mirror))
     )
-    (fp_text user %V (at 5.7 7.9) (layer F.SilkS)
+    (fp_text user %V (at 5.7 7.9 90) (layer F.SilkS)
       (effects (font (size 1 1) (thickness 0.15)))
     )
@@
     (fp_line (start -5.48 3.645) (end -5.48 -1.105) (layer B.SilkS) (width 0.12))
     (fp_line (start 15.37 2.295) (end 15.37 -1.105) (layer B.SilkS) (width 0.12))
-    (pad R thru_hole circle (at 6.35 0) (size 3.2 3.2) (drill 1.7) (layers *.Cu *.Mask)
+    (pad R thru_hole circle (at 6.35 0 90) (size 3.2 3.2) (drill 1.7) (layers *.Cu *.Mask)
       (net 28 "Net-(J2-PadR)"))
-    (pad S thru_hole circle (at 12.7 0) (size 3.2 3.2) (drill 1.7) (layers *.Cu *.Mask)
-      (net 7 GND))
-    (pad T thru_hole circle (at 0 0) (size 3.2 3.2) (drill 1.7) (layers *.Cu *.Mask)
+    (pad S thru_hole circle (at 12.7 0 90) (size 3.2 3.2) (drill 1.7) (layers *.Cu *.Mask)
+      (net 7 GND))
+    (pad T thru_hole circle (at 0 0 90) (size 3.2 3.2) (drill 1.7) (layers *.Cu *.Mask)
       (net 29 JACK_OUT))
-    (pad RN thru_hole circle (at 6.35 16.23) (size 3.2 3.2) (drill 1.7) (layers *.Cu *.Mask)
+    (pad RN thru_hole circle (at 6.35 16.23 90) (size 3.2 3.2) (drill 1.7) (layers *.Cu *.Mask)
       (net 30 "Net-(J2-PadRN)"))
-    (pad SN thru_hole circle (at 12.7 16.23) (size 3.2 3.2) (drill 1.7) (layers *.Cu *.Mask)
-      (net 7 GND))
-    (pad TN thru_hole circle (at 0 16.23) (size 3.2 3.2) (drill 1.7) (layers *.Cu *.Mask)
+    (pad SN thru_hole circle (at 12.7 16.23 90) (size 3.2 3.2) (drill 1.7) (layers *.Cu *.Mask)
+      (net 7 GND))
+    (pad TN thru_hole circle (at 0 16.23 90) (size 3.2 3.2) (drill 1.7) (layers *.Cu *.Mask)
       (net 31 "Net-(J2-PadTN)"))
     (model ${KISYS3DMOD}/Connector_Audio.3dshapes/Jack_6.35mm_Neutrik_NMJ6HCD3_Horizontal.wrl
@@
   )
   (module pedal-component-footprint:Jack_6.35mm_Neutrik_NMJ6HCD3_Horizontal (layer F.Cu)
-    (at -79.2172 117.5408)
+    (at 64 73.5 90)
     (descr "M Series, 6.35mm (1/4in) stereo jack, switched, with chrome ferrule and offset PCB pins, https://www.neutrik.com/en/product/nmj6hcd3")
     (tags "neutrik jack m")
-    (fp_text reference J1 (at 6.35 6.0325) (layer F.Fab)
-      (effects (font (size 1 1) (thickness 0.15)))
-    )
-    (fp_text value IN (at 5.3975 7.874) (layer B.SilkS)
+    (fp_text reference J1 (at 6.35 6.0325 90) (layer F.Fab)
+      (effects (font (size 1 1) (thickness 0.15)))
+    )
+    (fp_text value IN (at 5.3975 7.874 90) (layer B.SilkS)
       (effects (font (size 1 1) (thickness 0.15)) (justify mirror))
     )
-    (fp_text user %V (at 5.7 7.9) (layer F.SilkS)
+    (fp_text user %V (at 5.7 7.9 90) (layer F.SilkS)
       (effects (font (size 1 1) (thickness 0.15)))
     )
@@
     (fp_line (start -5.48 3.645) (end -5.48 -1.105) (layer B.SilkS) (width 0.12))
     (fp_line (start 15.37 2.295) (end 15.37 -1.105) (layer B.SilkS) (width 0.12))
-    (pad R thru_hole circle (at 6.35 0) (size 3.2 3.2) (drill 1.7) (layers *.Cu *.Mask)
+    (pad R thru_hole circle (at 6.35 0 90) (size 3.2 3.2) (drill 1.7) (layers *.Cu *.Mask)
       (net 24 "Net-(J1-PadR)"))
-    (pad S thru_hole circle (at 12.7 0) (size 3.2 3.2) (drill 1.7) (layers *.Cu *.Mask)
-      (net 7 GND))
-    (pad T thru_hole circle (at 0 0) (size 3.2 3.2) (drill 1.7) (layers *.Cu *.Mask)
+    (pad S thru_hole circle (at 12.7 0 90) (size 3.2 3.2) (drill 1.7) (layers *.Cu *.Mask)
+      (net 7 GND))
+    (pad T thru_hole circle (at 0 0 90) (size 3.2 3.2) (drill 1.7) (layers *.Cu *.Mask)
       (net 25 JACK_IN))
-    (pad RN thru_hole circle (at 6.35 16.23) (size 3.2 3.2) (drill 1.7) (layers *.Cu *.Mask)
+    (pad RN thru_hole circle (at 6.35 16.23 90) (size 3.2 3.2) (drill 1.7) (layers *.Cu *.Mask)
       (net 26 "Net-(J1-PadRN)"))
-    (pad SN thru_hole circle (at 12.7 16.23) (size 3.2 3.2) (drill 1.7) (layers *.Cu *.Mask)
-      (net 7 GND))
-    (pad TN thru_hole circle (at 0 16.23) (size 3.2 3.2) (drill 1.7) (layers *.Cu *.Mask)
+    (pad SN thru_hole circle (at 12.7 16.23 90) (size 3.2 3.2) (drill 1.7) (layers *.Cu *.Mask)
+      (net 7 GND))
+    (pad TN thru_hole circle (at 0 16.23 90) (size 3.2 3.2) (drill 1.7) (layers *.Cu *.Mask)
       (net 27 "Net-(J1-PadTN)"))
     (model ${KISYS3DMOD}/Connector_Audio.3dshapes/Jack_6.35mm_Neutrik_NMJ6HCD3_Horizontal.wrl

Commit message: Edge cuts done
Parts:
- moved RV3 1.90 mm to (147.2, 67.8)
Other:
- board outline added: 110 x 84 mm
- net class Power added: clearance 0.25, trace_width 0.35, via_dia 0.8, via_drill 0.4
Changed lines of the file:
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@@
   (general
     (thickness 1.6)
-    (drawings 0)
+    (drawings 20)
     (tracks 0)
     (zones 0)
@@
     (uvia_dia 0.3)
     (uvia_drill 0.1)
-    (add_net +4V5)
-    (add_net +9V)
-    (add_net CI)
-    (add_net CV)
     (add_net FLIP_IN1)
     (add_net FLIP_IN2)
@@
     (add_net FX_SEND1)
     (add_net FX_SEND2)
-    (add_net GND)
     (add_net IN)
     (add_net JACK_IN)
@@
     (add_net OUT)
   )
+  (net_class Power ""
+    (clearance 0.25)
+    (trace_width 0.35)
+    (via_dia 0.8)
+    (via_drill 0.4)
+    (uvia_dia 0.3)
+    (uvia_drill 0.1)
+    (add_net +4V5)
+    (add_net +9V)
+    (add_net CI)
+    (add_net CV)
+    (add_net GND)
+  )
   (module "MBv3 enclosures:1590BB" (layer F.Cu)
     (at 100 100 90)
@@
   )
   (module "MBv3 potentiometers:16MM_B.MOUNT" (layer F.Cu)
-    (at 149 68.5 90)
+    (at 147.25 67.75 90)
     (descr "<b>16mm / Right-Angle /  PC Mount / Short Pin</b>\n<p>\nFor bottom-mount potentiometers\n<p>\n<a href=\"http://smallbear-electronics.mybigcommerce.com/alpha-single-gang-16mm-right-angle-pc-mount/\">http://smallbear-electronics.mybigcommerce.com/alpha-single-gang-16mm-right-angle-pc-mount/</a>")
     (fp_text reference RV3 (at 0 -2.413 90) (layer B.SilkS)
@@
       (net 2 IN))
   )
+  (gr_line (start 117.5 58) (end 149 58) (layer Edge.Cuts) (width 0.05))
+  (gr_line (start 51 58) (end 103.25 58) (layer Edge.Cuts) (width 0.05))
+  (gr_arc (start 115.5 74.25) (end 115.5 75.25) (angle -90) (layer Edge.Cuts) (width 0.05))
+  (gr_arc (start 105.25 74.25) (end 104.25 74.25) (angle -90) (layer Edge.Cuts) (width 0.05))
+  (gr_arc (start 103.25 59) (end 104.25 59) (angle -90) (layer Edge.Cuts) (width 0.05))
+  (gr_arc (start 117.5 59) (end 117.5 58) (angle -90) (layer Edge.Cuts) (width 0.05))
+  (gr_line (start 116.5 74.25) (end 116.5 59) (layer Edge.Cuts) (width 0.05))
+  (gr_line (start 105.25 75.25) (end 115.5 75.25) (layer Edge.Cuts) (width 0.05))
+  (gr_line (start 104.25 59) (end 104.25 74.25) (layer Edge.Cuts) (width 0.05))
+  (gr_arc (start 45 58) (end 45 64) (angle -90) (layer Edge.Cuts) (width 0.05))
+  (gr_arc (start 155 58) (end 149 58) (angle -90) (layer Edge.Cuts) (width 0.05))
+  (gr_arc (start 152 124.5) (end 152 127.5) (angle -90) (layer Edge.Cuts) (width 0.05))
+  (gr_arc (start 122.25 130.5) (end 122.25 127.5) (angle -90) (layer Edge.Cuts) (width 0.05))
+  (gr_arc (start 116.25 139) (end 116.25 142) (angle -90) (layer Edge.Cuts) (width 0.05))
+  (gr_line (start 119.25 139) (end 119.25 130.5) (layer Edge.Cuts) (width 0.05))
+  (gr_line (start 122.25 127.5) (end 152 127.5) (layer Edge.Cuts) (width 0.05))
+  (gr_arc (start 45 142) (end 51 142) (angle -90) (layer Edge.Cuts) (width 0.05))
+  (gr_line (start 116.25 142) (end 51 142) (layer Edge.Cuts) (width 0.05))
+  (gr_line (start 155 64) (end 155 124.5) (layer Edge.Cuts) (width 0.05))
+  (gr_line (start 45 136) (end 45 64) (layer Edge.Cuts) (width 0.05))
 )

Commit message: Power section
Parts:
- moved H4 156.8 mm to (109.5, 77.1)
- moved D3 155.7 mm to (115.9, 82.2), turned to 180 degrees
- moved H3 149.2 mm to (112.1, 77.1)
- moved R23 132.9 mm to (93.4, 84.8)
- moved C7 118.2 mm to (113.3, 87.3), turned to 180 degrees
- moved R22 115.6 mm to (93.4, 87.3), turned to 180 degrees
- moved C8 108.2 mm to (103.2, 87.3)
Changed lines of the file:
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@@
     (aux_axis_origin 0 0)
     (grid_origin 100 100)
-    (visible_elements FFFFF77F)
+    (visible_elements FFFFFF7F)
     (pcbplotparams
       (layerselection 0x010fc_ffffffff)
@@
   )
   (module "MBv3 resistors:0.3_22.B" (layer F.Cu)
-    (at -35.732201 116.098)
+    (at 93.396 84.76)
     (descr "0.3\"  (7.62mm) lead spacing, 1/4W (flat)")
     (fp_text reference R23 (at 0 0) (layer F.SilkS)
@@
   )
   (module "MBv3 resistors:0.3_22.B" (layer F.Cu)
-    (at -21.822201 96.628)
+    (at 93.396 87.3 180)
     (descr "0.3\"  (7.62mm) lead spacing, 1/4W (flat)")
     (fp_text reference R22 (at 0 0) (layer F.SilkS)
@@
     (fp_arc (start -2.556 0.762) (end -2.81 0.762) (angle -90) (layer F.SilkS) (width 0.1524))
     (fp_arc (start -2.556 -0.762) (end -2.81 -0.762) (angle 90) (layer F.SilkS) (width 0.1524))
-    (pad 2 thru_hole oval (at 3.81 0) (size 2 2) (drill 1) (layers *.Cu *.Mask)
+    (pad 2 thru_hole oval (at 3.81 0 180) (size 2 2) (drill 1) (layers *.Cu *.Mask)
       (net 14 +4V5))
-    (pad 1 thru_hole oval (at -3.81 0) (size 2 2) (drill 1) (layers *.Cu *.Mask)
+    (pad 1 thru_hole oval (at -3.81 0 180) (size 2 2) (drill 1) (layers *.Cu *.Mask)
       (net 13 +9V))
     (model ${KISYS3DMOD}/Resistor_THT.3dshapes/R_Axial_DIN0207_L6.3mm_D2.5mm_P7.62mm_Horizontal.wrl
@@
   )
   (module pedal-component-footprint:PinHeader_1x01_P2.54mm_Vertical_Front_Back (layer F.Cu)
-    (at -38.9922 127.5223)
+    (at 109.525 77.14)
     (descr "Through hole straight pin header, 1x01, 2.54mm pitch, single row")
     (tags "Through hole pin header THT 1x01 2.54mm single row")
@@
   )
   (module pedal-component-footprint:PinHeader_1x01_P2.54mm_Vertical_Front_Back (layer F.Cu)
-    (at -30.9822 119.5123)
+    (at 112.065 77.14)
     (descr "Through hole straight pin header, 1x01, 2.54mm pitch, single row")
     (tags "Through hole pin header THT 1x01 2.54mm single row")
@@
   )
   (module Diode_THT:D_DO-41_SOD81_P10.16mm_Horizontal (layer F.Cu)
-    (at -39.1672 96.4808)
+    (at 115.875 82.22 180)
     (descr "Diode, DO-41_SOD81 series, Axial, Horizontal, pin pitch=10.16mm, , length*diameter=5.2*2.7mm^2, , http://www.diodes.com/_files/packages/DO-41%20(Plastic).pdf")
     (tags "Diode DO-41_SOD81 series Axial Horizontal pin pitch 10.16mm  length 5.2mm diameter 2.7mm")
-    (fp_text reference D3 (at 5.08 -2.47) (layer F.SilkS)
+    (fp_text reference D3 (at 6.985 -2.47) (layer F.SilkS)
       (effects (font (size 1 1) (thickness 0.15)))
     )
@@
     (fp_line (start 2.48 1.35) (end 7.68 1.35) (layer F.Fab) (width 0.1))
     (fp_line (start 2.48 -1.35) (end 2.48 1.35) (layer F.Fab) (width 0.1))
-    (pad 2 thru_hole oval (at 10.16 0) (size 2.2 2.2) (drill 1.1) (layers *.Cu *.Mask)
-      (net 7 GND))
-    (pad 1 thru_hole rect (at 0 0) (size 2.2 2.2) (drill 1.1) (layers *.Cu *.Mask)
+    (pad 2 thru_hole oval (at 10.16 0 180) (size 2.2 2.2) (drill 1.1) (layers *.Cu *.Mask)
+      (net 7 GND))
+    (pad 1 thru_hole rect (at 0 0 180) (size 2.2 2.2) (drill 1.1) (layers *.Cu *.Mask)
       (net 13 +9V))
     (model ${KISYS3DMOD}/Diode_THT.3dshapes/D_DO-41_SOD81_P10.16mm_Horizontal.wrl
@@
   )
   (module "MBv3 caps-elec:0504" (layer F.Cu)
-    (at -4.902201 81.662)
+    (at 103.175 87.3)
     (descr "0.2\" (5.08mm) spacing")
-    (fp_text reference C8 (at 0 0) (layer F.Fab)
+    (fp_text reference C8 (at 0 0) (layer F.SilkS)
       (effects (font (size 1.2065 1.2065) (thickness 0.1524)))
     )
-    (fp_text value 47u (at 0 0) (layer F.SilkS)
+    (fp_text value 47u (at 0 0) (layer F.SilkS) hide
       (effects (font (size 1.524 1.524) (thickness 0.15)))
     )
@@
   )
   (module "MBv3 caps-elec:0633" (layer F.Cu)
-    (at -4.902201 88.462)
+    (at 113.335 87.3 180)
     (descr "0.2\" (5.08mm) spacing")
     (fp_text reference C7 (at 0 0) (layer F.SilkS)
       (effects (font (size 0.9652 0.9652) (thickness 0.12192)))
     )
-    (fp_text value 100u (at 0 0) (layer F.SilkS)
+    (fp_text value 100u (at 0 0) (layer F.SilkS) hide
       (effects (font (size 1.524 1.524) (thickness 0.15)))
     )
@@
     (fp_line (start -1.778 -2.1844) (end -1.778 -1.5494) (layer F.SilkS) (width 0.1524))
     (fp_circle (center 0 0) (end 3.15 0) (layer F.SilkS) (width 0.1524))
-    (pad 2 thru_hole oval (at 2.54 0) (size 2 2) (drill 1) (layers *.Cu *.Mask)
-      (net 7 GND))
-    (pad 1 thru_hole rect (at -2.54 0) (size 2 2) (drill 1) (layers *.Cu *.Mask)
+    (pad 2 thru_hole oval (at 2.54 0 180) (size 2 2) (drill 1) (layers *.Cu *.Mask)
+      (net 7 GND))
+    (pad 1 thru_hole rect (at -2.54 0 180) (size 2 2) (drill 1) (layers *.Cu *.Mask)
       (net 13 +9V))
   )
