File: ab-mix/ab-mix.kicad_pcb (KiCad board)
At the start: 2 copper layers, 110 x 84 mm, 70 parts, among them J1 IN, J2 Out, J3 Send1, J4 Return1, J5 Send2, J6 Return2, J7 Exp, Q1 J201, Q2 J201, Q3 Q_PNP_EBC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

Commit message: Gerbers generated
Other:
- board text added: "JLCJLCJLCJLC"
- board text added: "weather changes v1.0 by @flpvsk"
Changed lines of the file:
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@@
   (general
     (thickness 1.6)
-    (drawings 20)
+    (drawings 22)
     (tracks 539)
     (zones 0)
@@
     (at 114.097 119.939 270)
     (descr "0.2\" (5.08mm) spacing")
-    (fp_text reference C4 (at 0 0 90) (layer F.Fab)
+    (fp_text reference C4 (at 0 0 90) (layer F.SilkS)
       (effects (font (size 1.2065 1.2065) (thickness 0.1524)))
     )
-    (fp_text value 10u (at 0 0 90) (layer F.SilkS)
+    (fp_text value 10u (at 0 0 90) (layer F.SilkS) hide
       (effects (font (size 1.524 1.524) (thickness 0.15)))
     )
@@
       (net 4 "Net-(C2-Pad1)"))
   )
+  (gr_text JLCJLCJLCJLC (at 47.752 128.016 90) (layer F.SilkS)
+    (effects (font (size 1 1) (thickness 0.15)))
+  )
+  (gr_text "weather changes\nv1.0\nby @flpvsk" (at 153.924 123.444) (layer F.SilkS)
+    (effects (font (size 1 1) (thickness 0.15)) (justify right))
+  )
   (gr_line (start 117.5 58) (end 149 58) (layer Edge.Cuts) (width 0.05))
